File: pcb/stepbuffer1.sch (KiCad schematic (older format))
At the start: 5 parts, among them J1 Conn_02x03_Odd_Even, P1 MA08-1, P2 MA08-1, U1 SN74LV4T125

Commit message: Update documentation
Parts:
- P1, P2: symbol SilentStepStick-TMC5160_v14-eagle-import:PINHD-1X08_2.54-S -> stepbuffer1-rescue:PINHD-1X08_2.54-S-SilentStepStick-TMC5160_v14-eagle-import
Changed lines of the file:
@@
 DCO
 $Comp
-L SilentStepStick-TMC5160_v14-eagle-import:GND #GND010
+L stepbuffer1-rescue:GND-SilentStepStick-TMC5160_v14-eagle-import #GND010
 U 1 1 845C69E3
 P 2200 7300
@@
 $EndComp
 $Comp
-L SilentStepStick-TMC5160_v14-eagle-import:PINHD-1X08_2.54-S P1
+L stepbuffer1-rescue:PINHD-1X08_2.54-S-SilentStepStick-TMC5160_v14-eagle-import P1
 U 1 1 D245C58C
 P 1850 4850
@@
 $EndComp
 $Comp
-L SilentStepStick-TMC5160_v14-eagle-import:PINHD-1X08_2.54-S P2
+L stepbuffer1-rescue:PINHD-1X08_2.54-S-SilentStepStick-TMC5160_v14-eagle-import P2
 U 1 1 2560E369
 P 1850 6700
@@
 	4350 6100 4650 6100
 $Comp
-L SilentStepStick-TMC5160_v14-eagle-import:GND #GND0101
+L stepbuffer1-rescue:GND-SilentStepStick-TMC5160_v14-eagle-import #GND0101
 U 1 1 5E22436D
 P 4700 7250
