File: pcb/stepbuffer1.kicad_pcb (KiCad board)
At the start: 2 copper layers, 15.2 x 20.3 mm, 5 parts, among them J1 Conn_02x03_Odd_Even, P1 MA08-1, P2 MA08-1, U1 SN74LV4T125

Commit message: Add all additional files Add additional board prototype for a plug-in to screw terminal board
Other:
- board text added: "D"
- board text added: "E"
- board text added: "G"
- board text added: "M"
- board text added: "S"
- board text added: "V"
- board text removed: "BMA1"
- board text removed: "BMA2"
- board text removed: "BMB1"
- board text removed: "BMB2"
- board text removed: "CSN/CFG3"
- board text removed: "DCO"
- board text removed: "Dir"
- board text removed: "EN"
- board text removed: "GND"
- board text removed: "SCK/CFG2"
- board text removed: "SDI/CFG1"
- board text removed: "SDO/CFG0"
- board text removed: "Step"
- board text removed: "Vio"
- board text removed: "Vm"
Changed lines of the file:
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@@
   (general
     (thickness 1.6)
-    (drawings 20)
+    (drawings 16)
     (tracks 78)
     (zones 0)
@@
       (net 1 GND))
   )
+  (gr_text G (at 153.01 113.91) (layer B.SilkS)
+    (effects (font (size 1 1) (thickness 0.15)) (justify mirror))
+  )
+  (gr_text S (at 153.07 106.3) (layer F.SilkS)
+    (effects (font (size 1 1) (thickness 0.15)))
+  )
+  (gr_text D (at 153.07 108.8) (layer F.SilkS)
+    (effects (font (size 1 1) (thickness 0.15)))
+  )
+  (gr_text E (at 153.07 103.83) (layer F.SilkS)
+    (effects (font (size 1 1) (thickness 0.15)))
+  )
+  (gr_text G (at 153.1 101.25) (layer F.SilkS)
+    (effects (font (size 1 1) (thickness 0.15)))
+  )
+  (gr_text M (at 152.99 96.07) (layer F.SilkS)
+    (effects (font (size 1 1) (thickness 0.15)))
+  )
+  (gr_text G (at 153.07 98.61) (layer F.SilkS)
+    (effects (font (size 1 1) (thickness 0.15)))
+  )
+  (gr_text V (at 153.28 111.47) (layer F.SilkS)
+    (effects (font (size 1 1) (thickness 0.15)))
+  )
+  (gr_text G (at 153.13 113.94) (layer F.SilkS)
+    (effects (font (size 1 1) (thickness 0.15)))
+  )
+  (gr_text E (at 143.81 96.15) (layer F.SilkS)
+    (effects (font (size 1 1) (thickness 0.15)))
+  )
+  (gr_text D (at 144 113.9) (layer F.SilkS)
+    (effects (font (size 1 1) (thickness 0.15)))
+  )
+  (gr_text S (at 143.89 111.42) (layer F.SilkS)
+    (effects (font (size 1 1) (thickness 0.15)))
+  )
   (gr_line (start 140.8811 115.1636) (end 156.1211 115.1636) (layer Edge.Cuts) (width 0.05))
   (gr_line (start 156.1211 115.1636) (end 156.1211 94.8436) (layer Edge.Cuts) (width 0.05))
   (gr_line (start 156.1211 94.8436) (end 140.8811 94.8436) (layer Edge.Cuts) (width 0.05))
   (gr_line (start 140.8811 94.8436) (end 140.8811 115.1636) (layer Edge.Cuts) (width 0.05))
-  (gr_text GND (at 156.7561 96.7486) (layer Cmts.User)
-    (effects (font (size 1.2065 1.2065) (thickness 0.1651)) (justify left bottom))
-  )
-  (gr_text Vio (at 156.7561 99.2886) (layer Cmts.User)
-    (effects (font (size 1.2065 1.2065) (thickness 0.1651)) (justify left bottom))
-  )
-  (gr_text BMB2 (at 156.7561 101.8286) (layer Cmts.User)
-    (effects (font (size 1.2065 1.2065) (thickness 0.1651)) (justify left bottom))
-  )
-  (gr_text BMB1 (at 156.7561 104.3686) (layer Cmts.User)
-    (effects (font (size 1.2065 1.2065) (thickness 0.1651)) (justify left bottom))
-  )
-  (gr_text BMA1 (at 156.7561 106.9086) (layer Cmts.User)
-    (effects (font (size 1.2065 1.2065) (thickness 0.1651)) (justify left bottom))
-  )
-  (gr_text BMA2 (at 156.7561 109.4486) (layer Cmts.User)
-    (effects (font (size 1.2065 1.2065) (thickness 0.1651)) (justify left bottom))
-  )
-  (gr_text GND (at 156.7561 111.9886) (layer Cmts.User)
-    (effects (font (size 1.2065 1.2065) (thickness 0.1651)) (justify left bottom))
-  )
-  (gr_text Vm (at 156.7561 114.5286) (layer Cmts.User)
-    (effects (font (size 1.2065 1.2065) (thickness 0.1651)) (justify left bottom))
-  )
-  (gr_text EN (at 140.2461 113.2586) (layer Cmts.User)
-    (effects (font (size 1.2065 1.2065) (thickness 0.1651)) (justify right top))
-  )
-  (gr_text SDI/CFG1 (at 140.2461 110.7186) (layer Cmts.User)
-    (effects (font (size 1.2065 1.2065) (thickness 0.1651)) (justify right top))
-  )
-  (gr_text SCK/CFG2 (at 140.2461 108.1786) (layer Cmts.User)
-    (effects (font (size 1.2065 1.2065) (thickness 0.1651)) (justify right top))
-  )
-  (gr_text CSN/CFG3 (at 140.2461 105.6386) (layer Cmts.User)
-    (effects (font (size 1.2065 1.2065) (thickness 0.1651)) (justify right top))
-  )
-  (gr_text SDO/CFG0 (at 140.2461 103.0986) (layer Cmts.User)
-    (effects (font (size 1.2065 1.2065) (thickness 0.1651)) (justify right top))
-  )
-  (gr_text DCO (at 140.2461 100.5586) (layer Cmts.User)
-    (effects (font (size 1.2065 1.2065) (thickness 0.1651)) (justify right top))
-  )
-  (gr_text Step (at 140.2461 98.0186) (layer Cmts.User)
-    (effects (font (size 1.2065 1.2065) (thickness 0.1651)) (justify right top))
-  )
-  (gr_text Dir (at 140.2461 95.4786) (layer Cmts.User)
-    (effects (font (size 1.2065 1.2065) (thickness 0.1651)) (justify right top))
-  )
   (segment (start 154.3203 99.2047) (end 154.851 98.674) (width 0.25) (layer Bottom) (net 1))
   (segment (start 149.7153 100.33) (end 149.7153 100.0486) (width 0.25) (layer Bottom) (net 1))
